Commit message: Added differential driver for two wheels

File: description/robot.urdf.xacro (robot description, xacro)
@@ -2,3 +2,4 @@
 <robot xmlns:xacro="http://www.ros.org/wiki/xacro"  name="robot">
     <xacro:include filename="robot_core.xacro"/>
+    <xacro:include filename="gazebo_control.xacro"/>
 </robot>

File: description/robot_core.xacro (robot description, xacro)
@@ -22,5 +22,5 @@
         <parent link="base_link"/>
         <child link="chassis"/>
-        <origin xyz="-0.1125 0 0"/>
+        <origin xyz="-0.09 0 0"/>
     </joint>
     <link name="chassis">
@@ -28,10 +28,10 @@
             <origin xyz="0.1125 0 0.055"/>
             <geometry>
-                <box size="0.225 0.215 0.11"/>
+                <box size="0.225 0.145 0.11"/>
             </geometry>
-            <material name="white"/>
+            <material name="red"/>
         </visual>
-        <xacro:inertial_box mass="0.5" x="0.225" y="0.3" z="0.15">
-            <origin xyz="0.15 0 0.075"/>
+        <xacro:inertial_box mass="0.5" x="0.225" y="0.145" z="0.11">
+            <origin xyz="0.1125 0 0.055"/>
         </xacro:inertial_box>
         <collision>
@@ -42,8 +42,11 @@
         </collision>
     </link>
+    <gazebo reference="chassis">
+            <material>Gazebo/White</material>
+    </gazebo>
     <joint name="left_wheel_joint" type="continuous">
         <parent link="base_link"/>
         <child link="left_wheel"/>
-        <origin xyz="0 0.1075 0" rpy="-${pi/2} 0 0"/>
+        <origin xyz="0 0.087 0" rpy="-${pi/2} 0 0"/>
         <axis xyz="0 0 1"/>
     </joint>
@@ -61,11 +64,14 @@
         </collision>
         <xacro:inertial_cylinder mass="0.1" length="0.017" radius="0.035">
-            <origin xyz="0.15 0 0.075" rpy="0 0 0"/>
+            <origin xyz="0 0 0" rpy="0 0 0"/>
         </xacro:inertial_cylinder>
     </link>
+     <gazebo reference="left_wheel">
+            <material>Gazebo/Black</material>
+    </gazebo>
     <joint name="right_wheel_joint" type="continuous">
         <parent link="base_link"/>
         <child link="right_wheel"/>
-        <origin xyz="0 -0.1075 0" rpy="${pi/2} 0 0"/>
+        <origin xyz="0 -0.087 0" rpy="${pi/2} 0 0"/>
         <axis xyz="0 0 -1"/>
     </joint>
@@ -82,4 +88,37 @@
             </geometry>
         </collision>
+        <xacro:inertial_cylinder mass="0.1" length="0.017" radius="0.035">
+            <origin xyz="0 0 0" rpy="0 0 0"/>
+        </xacro:inertial_cylinder>
     </link>
+     <gazebo reference="right_wheel">
+            <material>Gazebo/Black</material>
+    </gazebo>
+    <joint name="caster_wheel_joint" type="fixed">
+        <parent link="chassis"/>
+        <child link="caster_wheel"/>
+        <origin xyz="0.14 0 0"/>
+    </joint>
+    <link name="caster_wheel">
+        <visual>
+            <geometry>
+                <sphere radius="0.035"/>
+            </geometry>
+            <material name="black"/>
+        </visual>
+        <collision>
+            <geometry>
+                <sphere radius="0.035"/>
+            </geometry>
+            <material name="black"/>
+        </collision>
+        <xacro:inertial_sphere mass="0.1" radius="0.035">
+            <origin xyz="0 0 0" rpy="0 0 0"/>
+        </xacro:inertial_sphere>
+    </link>
+    <gazebo reference="caster_wheel">
+            <material>Gazebo/Silver</material>
+            <mu1 value="0.001"/>
+            <mu2 value="0.001"/>
+    </gazebo>
 </robot>
