Commit message: Pushing four wheels

File: description/gazebo_control.xacro (robot description, xacro)
@@ -3,8 +3,11 @@
     <gazebo>
         <plugin name="diff_drive" filename="libgazebo_ros_diff_drive.so">
+            <num_wheel_pairs>2</num_wheel_pairs>
             <!-- Wheel Information -->
             <left_joint>left_wheel_joint</left_joint>
+            <left_joint>left_wheel_joint_b</left_joint>
             <right_joint>right_wheel_joint</right_joint>
-            <wheel_separation>0.35</wheel_separation>
+            <right_joint>right_wheel_joint_b</right_joint>
+            <wheel_separation>0.174</wheel_separation>
             <wheel_diameter>0.07</wheel_diameter>
             <!-- Performance Properties -->

File: description/robot_core.xacro (robot description, xacro)
@@ -48,5 +48,5 @@
         <parent link="base_link"/>
         <child link="left_wheel"/>
-        <origin xyz="0 0.087 0" rpy="-${pi/2} 0 0"/>
+        <origin xyz="0.08 0.087 0" rpy="-${pi/2} 0 0"/>
         <axis xyz="0 0 1"/>
     </joint>
@@ -73,5 +73,5 @@
         <parent link="base_link"/>
         <child link="right_wheel"/>
-        <origin xyz="0 -0.087 0" rpy="${pi/2} 0 0"/>
+        <origin xyz="0.08 -0.087 0" rpy="${pi/2} 0 0"/>
         <axis xyz="0 0 -1"/>
     </joint>
@@ -95,10 +95,60 @@
             <material>Gazebo/Black</material>
     </gazebo>
-    <joint name="caster_wheel_joint" type="fixed">
+    <joint name="left_wheel_joint_b" type="continuous">
+        <parent link="base_link"/>
+        <child link="left_wheel_b"/>
+        <origin xyz="-0.06 0.087 0" rpy="-${pi/2} 0 0"/>
+        <axis xyz="0 0 1"/>
+    </joint>
+    <link name="left_wheel_b">
+        <visual>
+            <geometry>
+                <cylinder radius="0.035" length="0.017"/>
+            </geometry>
+            <material name="black"/>
+        </visual>
+        <collision>
+            <geometry>
+                <cylinder radius="0.035" length="0.017"/>
+            </geometry>
+        </collision>
+        <xacro:inertial_cylinder mass="0.1" length="0.017" radius="0.035">
+            <origin xyz="0 0 0" rpy="0 0 0"/>
+        </xacro:inertial_cylinder>
+    </link>
+     <gazebo reference="left_wheel_b">
+            <material>Gazebo/Black</material>
+    </gazebo>
+    <joint name="right_wheel_joint_b" type="continuous">
+        <parent link="base_link"/>
+        <child link="right_wheel_b"/>
+        <origin xyz="-0.06 -0.087 0" rpy="${pi/2} 0 0"/>
+        <axis xyz="0 0 -1"/>
+    </joint>
+    <link name="right_wheel_b">
+        <visual>
+            <geometry>
+                <cylinder radius="0.035" length="0.017"/>
+            </geometry>
+            <material name="black"/>
+        </visual>
+        <collision>
+            <geometry>
+                <cylinder radius="0.035" length="0.017"/>
+            </geometry>
+        </collision>
+        <xacro:inertial_cylinder mass="0.1" length="0.017" radius="0.035">
+            <origin xyz="0 0 0" rpy="0 0 0"/>
+        </xacro:inertial_cylinder>
+    </link>
+     <gazebo reference="right_wheel_b">
+            <material>Gazebo/Black</material>
+    </gazebo>
+    <!-- <joint name="caster_wheel_joint" type="fixed">
         <parent link="chassis"/>
         <child link="caster_wheel"/>
         <origin xyz="0.14 0 0"/>
-    </joint>
-    <link name="caster_wheel">
+    </joint> -->
+    <!-- <link name="caster_wheel">
         <visual>
             <geometry>
@@ -121,4 +171,4 @@
             <mu1 value="0.001"/>
             <mu2 value="0.001"/>
-    </gazebo>
+    </gazebo> -->
 </robot>
